File: humep1.kicad_pcb (KiCad board)
At the start: 2 copper layers, 50 x 26.8 mm, 8 parts, among them U1 LM1117DT-3.3, U2 113991054

Commit message: updated schematic + completed pcb layout
Parts:
- removed JOY1: JOYSTICK_ANALOG_XY, JOYSTICK_ANALOG_MINITHM
- added JOYSTICK (2765): 2765, 2765:SW_2765, F.Cu at (46.7, 64.0)
- 1uF: renamed from C3; footprint Capacitor_SMD:C_0402_1005Metric_Pad0.74x0.62mm_HandSolder -> Capacitor_SMD:C_0805_2012Metric_Pad1.18x1.45mm_HandSolder
- moved 1uF 23.3 mm to (55.5, 76.5)
- moved 10uF 17.9 mm to (60.0, 61.3)
- moved 10uF 7.35 mm to (66.2, 61.3)
- moved U1 4.19 mm to (62.0, 70.1), turned to -90 degrees
- moved BATTERY 3.02 mm to (63.2, 57.0)
- moved 0.1uF 2.94 mm to (66.8, 67.5), turned to -90 degrees
- moved ESP32-C3 2.05 mm to (77.5, 64.0)
- renumbered C4 to 0.1uF, C1 to 10uF, C2 to 10uF, BT1 to BATTERY, U2 to ESP32-C3
Routing:
- net GND: track 0.00 -> 62.1 mm, vias 0 -> 4
- net /X: track 0.00 -> 56.2 mm
- net /Y: track 0.00 -> 42.6 mm
- net /3.3V: track 17.5 -> 42.4 mm, vias 1 -> 0
- net /PWR: track 33.6 -> 39.0 mm, vias 0 -> 2
- net (no net): track 0.98 -> 0.00 mm
Other:
- board size 50 x 26.8 mm -> 50 x 25.2 mm
- board text added: "+"
- board text added: "-"
- board text added: "3.3"
- board text added: "DX"
- board text added: "DY"
- board text added: "GND"
- board text added: "LM1117"
- board text added: "VI"
- board text added: "X:"
- board text added: "Y:"
- board text removed: "<-X"
- board text removed: "<-Y"
